File: kicad/MX-MAIN-C/MX-MAIN-C.kicad_sch (KiCad schematic)
At the start: 3 parts, among them U1 MC68000P, U2 MC6850

Commit message: kicad schematic updates
Parts:
- removed U3: ~, symbol oldcrapics:MC1488
- added A5: 74LS244, symbol 74xx:74LS244
- added A9: MC1488, symbol oldcrapics:MC1488
- added J1: DB25_Pins, symbol Connector:DB25_Pins
- added MJ2: Conn_02x05_Odd_Even, symbol Connector_Generic:Conn_02x05_Odd_Even
- added R1, R2, R3, US4, UT4: 74LS245, symbol 74xx:74LS245
- added R32: R, symbol Device:R
- added SW1: SW_DIP_x08, symbol Switch:SW_DIP_x08
- added U3: 74LS85, symbol 74xx:74LS85
- added UN2: 7417, symbol 74xx_IEEE:7417
Connections:
- net +12V: now also A9.14 (VCC+)
- net -12V: now also A9.1 (VCC-)
- net GND: now also U2.1 (VSS), A9.7 (GND), R32.2
- net at U1.1 (D4): now also US4.5 (A3)
- net at U1.17 (~{HALT}): now also UN2.6, UN2.9
- net at U1.18 (~{RESET}): now also UN2.11, UN2.4
- net at U1.2 (D3): now also US4.6 (A4)
- net at U1.29 (A1): now also R3.8 (A6)
- net at U1.3 (D2): now also US4.7 (A5)
- net at U1.30 (A2): now also R3.7 (A5)
- net at U1.31 (A3): now also R3.6 (A4)
- net at U1.32 (A4): now also R3.5 (A3)
- net at U1.33 (A5): now also R3.4 (A2)
- net at U1.34 (A6): now also R3.3 (A1)
- net at U1.35 (A7): now also R3.2 (A0)
- net at U1.36 (A8): now also R2.9 (A7)
- net at U1.37 (A9): now also R2.8 (A6)
- net at U1.38 (A10): now also R2.7 (A5)
- net at U1.39 (A11): now also R2.6 (A4)
- net at U1.4 (D1): now also US4.8 (A6)
- net at U1.40 (A12): now also R2.5 (A3)
- net at U1.41 (A13): now also R2.4 (A2)
- net at U1.42 (A14): now also R2.3 (A1)
- net at U1.43 (A15): now also R2.2 (A0)
- net at U1.44 (A16): now also R1.9 (A7)
- net at U1.45 (A17): now also R1.8 (A6)
- net at U1.46 (A18): now also R1.7 (A5)
- net at U1.47 (A19): now also R1.6 (A4)
- net at U1.48 (A20): now also R1.5 (A3)
- net at U1.5 (D0): now also US4.9 (A7)
- net at U1.50 (A21): now also R1.4 (A2)
- net at U1.51 (A22): now also R1.3 (A1)
- net at U1.52 (A23): now also R1.2 (A0)
- net at U1.54 (D15): now also UT4.2 (A0)
- net at U1.55 (D14): now also UT4.3 (A1)
- net at U1.56 (D13): now also UT4.4 (A2)
- net at U1.57 (D12): now also UT4.5 (A3)
- net at U1.58 (D11): now also UT4.6 (A4)
- net at U1.59 (D10): now also UT4.7 (A5)
- net at U1.60 (D9): now also UT4.8 (A6)
- net at U1.61 (D8): now also UT4.9 (A7)
- net at U1.62 (D7): now also US4.2 (A0)
- net at U1.63 (D6): now also US4.3 (A1)
- net at U1.64 (D5): now also US4.4 (A2)
- net acia_kb_txd: now reaches U2.6 (Tx_Data)
- net acia_kb_txd: now also A9.2 (1A)
- new net: R32.1, UN2.3, UN2.5
- new net: A5.11 (I0b), SW1.8
- new net: A5.13 (I1b), SW1.6
- new net: A5.6 (I2a), SW1.5
- new net: A5.8 (I3a), SW1.7
- new net: SW1.1, U3.9 (B0)
- new net: SW1.2, U3.11 (B1)
- new net: MJ2.1 (Pin_1), U3.1 (B3)
- new net character_txd: A9.3 (1Y), J1.9
Other:
- note added: "d2 pal pin 7"
- note added: "d2 pal pin 8 + other places, there are traces"
- note added: "j2 pin 11"
- moved on the sheet: U1, U2

Commit message: schematic updates
Parts:
- added U4: ~, symbol oldcrapics:GA040
- added UE2, UF2: 2764, Package_DIP:DIP-28_W15.24mm, symbol Memory_EPROM:2764
- added UK2: 74LS04, symbol 74xx:74LS04
- added UN1: 74LS244, symbol 74xx:74LS244
- added UP3: 74LS245, symbol 74xx:74LS245
- renumbered R1 to UR1, R2 to UR2, R3 to UR3
Connections:
- net GND: now also U4.20
- net at UT4.11 (B7): now also UF2.19 (D7)
- net at US4.11 (B7): now also UE2.11 (D0)
- net at US4.12 (B6): now also UE2.12 (D1)
- net at US4.13 (B5): now also UE2.13 (D2)
- net at US4.14 (B4): now also UE2.15 (D3)
- net at US4.15 (B3): now also UE2.16 (D4)
- net at US4.16 (B2): now also UE2.17 (D5)
- net at US4.17 (B1): now also UE2.18 (D6)
- net at US4.18 (B0): now also UE2.19 (D7)
- net at UR2.11 (B7): now also UE2.3 (A7), UF2.3 (A7)
- net at UR2.12 (B6): now also UE2.25 (A8), UF2.25 (A8)
- net at UR2.13 (B5): now also UE2.24 (A9), UF2.24 (A9)
- net at UR2.14 (B4): now also UE2.21 (A10), UF2.21 (A10)
- net at UR2.15 (B3): now also UE2.23 (A11), UF2.23 (A11)
- net at UR2.16 (B2): now also UE2.2 (A12), UF2.2 (A12)
- net at U1.22 (~{BERR}): now also UN1.18 (O0a)
- net at UR3.12 (B6): now also UR3.14 (B4), UR3.16 (B2), UR3.18 (B0), U4.1, U4.3, UE2.10 (A0), UE2.4 (A6), UE2.6 (A4), UE2.8 (A2), UF2.10 (A0), UF2.4 (A6), UF2.6 (A4), UF2.8 (A2), UP3.3 (A1), UP3.5 (A3), UP3.7 (A5), UP3.9 (A7)
- net at UR3.13 (B5): now also UR3.15 (B3), UR3.17 (B1), U4.2, UE2.5 (A5), UE2.7 (A3), UE2.9 (A1), UF2.5 (A5), UF2.7 (A3), UF2.9 (A1), UP3.4 (A2), UP3.6 (A4), UP3.8 (A6)
- new net: UK2.9, UN1.4 (I1a)
- new net: U4.15, UN1.2 (I0a)
- new net +5V: U4.40
Other:
- moved on the sheet: A5, MJ2, R32, SW1, U1, U3, UN2A, UN2B, UN2C, UN2D, UN2E, UN2F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

Commit message: kicad schematic update
Parts:
- added U4: GA042, symbol oldcrapics:GA042
- added U5: MC6845, Package_DIP:DIP-40_W15.24mm, symbol GPU:MC6845
- added U6: MC6840, Package_DIP:DIP-28_W15.24mm, symbol Interface:MC6840
- added UP1, UP2: 74LS670, symbol 74xx:74LS670
- UL3: renamed from U4; value ~ -> GA040
Connections:
- net +5V: now also U4.40
- net GND: now also U4.20
- net at UT4.1 (A->B): now also UK2.8, US4.1 (A->B)
- net buffered_d8: now reaches UF2.19 (D7), UT4.11 (B7)
- net buffered_d8: now also U5.33 (D0)
- net buffered_d9: now reaches UT4.12 (B6)
- net buffered_d9: now also U5.32 (D1)
- net buffered_d10: now reaches UT4.13 (B5)
- net buffered_d10: now also U5.31 (D2)
- net buffered_d11: now reaches UT4.14 (B4)
- net buffered_d11: now also U5.30 (D3)
- net buffered_d12: now reaches UT4.15 (B3)
- net buffered_d12: now also U5.29 (D4)
- net buffered_d13: now reaches UT4.16 (B2)
- net buffered_d13: now also U5.28 (D5)
- net buffered_d14: now reaches UT4.17 (B1)
- net buffered_d14: now also U5.27 (D6)
- net buffered_d15: now reaches UT4.18 (B0)
- net buffered_d15: now also U5.26 (D7)
- net at UT4.19 (CE): now also UL3.22, US4.19 (CE), U4.12
- net at UK2.9, UN1.4 (I1a): now also U1.9 (R/~{W})
- net at UR1.19 (CE): now also UR2.19 (CE), UR3.19 (CE)
- net buffered_a8: now reaches UE2.3 (A7), UF2.3 (A7), UR2.11 (B7)
- net buffered_a9: now reaches UE2.25 (A8), UF2.25 (A8), UR2.12 (B6)
- net buffered_a10: now reaches UE2.24 (A9), UF2.24 (A9), UR2.13 (B5)
- net buffered_a11: now reaches UE2.21 (A10), UF2.21 (A10), UR2.14 (B4)
- net buffered_a12: now reaches UE2.23 (A11), UF2.23 (A11), UR2.15 (B3)
- net buffered_a13: now reaches UE2.2 (A12), UF2.2 (A12), UR2.16 (B2)
- net buffered_a14: now reaches UR2.17 (B1)
- net buffered_a15: now reaches UR2.18 (B0)
- net rom_ce: now reaches UE2.20 (~{CE})
- net rom_ce: now also UF2.20 (~{CE}), U4.24
- net buffered_lds: now reaches UE2.22 (~{OE})
- net buffered_lds: now also UL3.34, UN1.7 (O1b), U4.14
- net buffered_uds: now reaches UF2.22 (~{OE})
- net buffered_uds: now also UL3.33, UN1.5 (O2b), U4.13
- net at UL3.6: now also U1.6 (~{AS}), UN1.17 (I3b)
- net at UN1.13 (I1b): now also U1.8 (~{LDS})
- net at UN1.14 (O2a): now also U1.10 (~{DTACK})
- net at UN1.15 (I2b): now also U1.7 (~{UDS})
- new net buffered_a1: U4.3, UE2.10 (A0), UF2.10 (A0), UL3.1, UP3.9 (A7), UR3.12 (B6)
- new net buffered_a2: U4.4, UE2.9 (A1), UF2.9 (A1), UL3.2, UP3.8 (A6), UR3.13 (B5)
- new net buffered_a3: UE2.8 (A2), UF2.8 (A2), UL3.3, UP3.7 (A5), UR3.14 (B4)
- new net buffered_a4: UE2.7 (A3), UF2.7 (A3), UP3.6 (A4), UR3.15 (B3)
- new net buffered_a5: UE2.6 (A4), UF2.6 (A4), UP3.5 (A3), UR3.16 (B2)
- new net buffered_a6: UE2.5 (A5), UF2.5 (A5), UP3.4 (A2), UR3.17 (B1)
- new net buffered_a7: UE2.4 (A6), UF2.4 (A6), UP3.3 (A1), UR3.18 (B0)
Other:
- moved on the sheet: UP3

Commit message: Update schematic
Parts:
- added UJ2: 74LS08, symbol 74xx:74LS08
Connections:
- net +5V: now also UP1.16 (VCC), UP2.16 (VCC)
- net GND: now also UP1.8 (GND), UP2.8 (GND)
- net buffered_d0: now reaches UE2.11 (D0), US4.11 (B7)
- net buffered_d0: now also UP2.15 (D1)
- net buffered_d1: now reaches UE2.12 (D1), US4.12 (B6)
- net buffered_d1: now also UP2.1 (D2)
- net buffered_d2: now reaches UE2.13 (D2), US4.13 (B5)
- net buffered_d2: now also UP2.2 (D3)
- net buffered_d3: now reaches UE2.15 (D3), US4.14 (B4)
- net buffered_d3: now also UP2.3 (D4)
- net buffered_d4: now reaches UE2.16 (D4), US4.15 (B3)
- net buffered_d4: now also UP1.15 (D1)
- net buffered_d5: now reaches UE2.17 (D5), US4.16 (B2)
- net buffered_d5: now also UP1.1 (D2)
- net buffered_d6: now reaches UE2.18 (D6), US4.17 (B1)
- net buffered_d6: now also UP1.2 (D3)
- net buffered_d7: now reaches UE2.19 (D7), US4.18 (B0)
- net buffered_d7: now also UP1.3 (D4)
- net buffered_a16: now reaches UR1.11 (B7)
- net buffered_a16: now also UP2.10 (Q1)
- net buffered_a17: now reaches UR1.12 (B6)
- net buffered_a17: now also UP2.9 (Q2)
- net buffered_a18: now reaches UR1.13 (B5)
- net buffered_a18: now also UP2.7 (Q3)
- net buffered_a19: now reaches UR1.14 (B4)
- net buffered_a19: now also UP2.6 (Q4)
- net buffered_a20: now reaches UR1.15 (B3)
- net buffered_a20: now also UP1.10 (Q1)
- net buffered_a21: now reaches UR1.16 (B2)
- net buffered_a21: now also UP1.9 (Q2)
- net buffered_a22: now reaches UR1.17 (B1)
- net buffered_a22: now also UP1.7 (Q3)
- net buffered_a23: now reaches UR1.18 (B0)
- net buffered_a23: now also UP1.6 (Q4)
- net at UP2.11 (~{Er}): now also UP1.11 (~{Er})
- net at UP2.12 (~{Ew}): now also UP1.12 (~{Ew})
- net at UP2.13 (Wb): now also UP1.13 (Wb)
- net at UP2.14 (Wa): now also UP1.14 (Wa)
- net at UP2.4 (Rb): now also UP1.4 (Rb), UJ2.11
- net at UP2.5 (Ra): now also UP1.5 (Ra), UJ2.3
Other:
- moved on the sheet: UP1, UP2

Commit message: schematic
Parts:
- added UN3: 8257, symbol oldcrapics:8257
- renumbered U6 to UH2, U4 to UL1
Connections:
- net buffered_a1: now also UP1.14 (Wa), UP2.14 (Wa)
- net buffered_a2: now also UP1.13 (Wb), UP2.13 (Wb)
- net buffered_d0: now also UN3.30 (D0)
- net buffered_d1: now also UN3.29 (D1)
- net buffered_d10: now also UF2.13 (D2)
- net buffered_d11: now also UF2.15 (D3)
- net buffered_d12: now also UF2.16 (D4)
- net buffered_d13: now also UF2.17 (D5)
- net buffered_d14: now also UF2.18 (D6)
- net buffered_d15: now also UF2.19 (D7)
- net buffered_d2: now also UN3.28 (D2)
- net buffered_d3: now also UN3.27 (D3)
- net buffered_d4: now also UN3.26 (D4)
- net buffered_d5: now also UN3.23 (D5)
- net buffered_d6: now also UN3.22 (D6)
- net buffered_d7: now also UN3.21 (D7)
- net buffered_d8: now also UF2.11 (D0); no longer UF2.19 (D7)
- net buffered_d9: now also UF2.12 (D1)
- net write: now reaches UK2.8, US4.1 (A->B), UT4.1 (A->B)
- net at UP1.11 (~{Er}), UP2.11 (~{Er}): now also UL1.34

Commit message: update schematic
Parts:
- added UJ3: 74LS155, symbol 74xx:74LS155
Connections:
- net buffered_a7: now also UJ3.13 (A0)
- net buffered_a8: now also UJ3.3 (A1)
- net buffered_a9: now also UJ3.1 (Ea1)
- net at UN3.11 (~{CS}): now also UJ3.7 (Q0a)
- net at U5.25 (~{CS}): now also UJ3.9 (Q0b)
- net at UL3.38: now also UJ3.5 (Q2a)
- net at UL1.26: now also UJ3.2 (Ea2)
- net at UL1.27: now also UJ3.15 (Eb2)
- net at UH2.15 (~{CS0}): now also UJ3.10 (Q1b)
Other:
- note added: "j111 graphics connector"

Commit message: update schematic
Parts:
- added YK3: CXO_DIP14, Oscillator:Oscillator_DIP-14, symbol Oscillator:CXO_DIP14
Connections:
- net GND: now also U1.16 (GND), U1.53 (GND)
- net at UL1.12, UL3.22, US4.19 (CE)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: now also UR1.19 (CE), UR2.19 (CE), UR3.19 (CE)
- net at UL3.19: now also U1.15 (CLK)
- net at UL3.7: now also YK3.8 (OUT)
- net at UL1.22: now also U1.28 (FC0)
- net at UL1.23: now also U1.27 (FC1)
Other:
- note added: "cn1"
